Commit message: Added YDLIDAR option as add-on

File: pmb2_description/robots/pmb2.urdf.xacro (robot description, xacro)
@@ -37,5 +37,5 @@
     <xacro:wrong_laser_model/>
   </xacro:if>
-  <xacro:if value="${add_on_module not in ['no-add-on', 'rgbd-sensors']}">
+  <xacro:if value="${add_on_module not in ['no-add-on', 'rgbd-sensors', 'lidar-back']}">
     <xacro:wrong_add_on_module/>
   </xacro:if>
@@ -51,4 +51,8 @@
   <xacro:if value="${add_on_module == 'rgbd-sensors'}">
     <xacro:include filename="$(find pmb2_description)/urdf/cameras_add_on/cameras_add_on.urdf.xacro" />
+  </xacro:if>
+  <!-- YDLIDAR TG15 mount -->
+  <xacro:if value="${add_on_module == 'lidar-back'}">
+    <xacro:include filename="$(find pmb2_description)/urdf/ydlidar_add_on/ydlidar_add_on.urdf.xacro" />
   </xacro:if>
   <!-- Materials for visualization -->
@@ -66,3 +70,7 @@
     <xacro:cameras_add_on name="cameras_add_on" parent="base_link"/>
   </xacro:if>
+  <!-- YDLIDAR TG15 Sensor -->
+  <xacro:if value="${add_on_module == 'lidar-back'}">
+    <xacro:ydlidar_add_on name="ydlidar" parent="base_link"/>
+  </xacro:if>
 </robot>

File: pmb2_description/urdf/base/base.urdf.xacro (robot description, xacro)
@@ -99,8 +99,8 @@
     <!-- Antennas -->
     <xacro:antenna name="${name}_antenna_left" parent="${name}_link">
-      <origin xyz="-0.201 0.1062 0.195" rpy="0 0 0"/>
+      <origin xyz="-0.186 0.135 0.195" rpy="0 0 0"/>
     </xacro:antenna>
     <xacro:antenna name="${name}_antenna_right" parent="${name}_link">
-      <origin xyz="-0.201 -0.1062 0.195" rpy="0 0 0"/>
+      <origin xyz="-0.186 -0.135 0.195" rpy="0 0 0"/>
     </xacro:antenna>
     <!-- Wheels -->

Commit message: Added lidar-back add-on to base configuration

File: pmb2_description/robots/pmb2.urdf.xacro (robot description, xacro)
@@ -21,5 +21,5 @@
   <xacro:arg name="has_microphone" default="false"/>
   <!-- false, true-->
-  <xacro:arg name="add_on_module" default="lidar-back"/>
+  <xacro:arg name="add_on_module" default="no-add-on"/>
   <!-- Execution env config -->
   <xacro:arg name="use_sim_time" default="false"/>

File: pmb2_description/urdf/base/base_sensors.urdf.xacro (robot description, xacro)
@@ -26,6 +26,7 @@
   <xacro:include filename="$(find pmb2_description)/urdf/sensors/range.urdf.xacro"/>
   <xacro:include filename="$(find pmb2_description)/urdf/sensors/microphone.urdf.xacro"/>
+  <xacro:include filename="$(find pmb2_description)/urdf/ydlidar_add_on/ydlidar_add_on.urdf.xacro" />
   <!-- MACRO DEFINITION -->
-  <xacro:macro name="base_sensors" params="name laser_model:=sick-571 has_sonars:=false has_microphone:=false" >
+  <xacro:macro name="base_sensors" params="name laser_model:=sick-571 has_sonars:=false has_microphone:=false add_on_module:=lidar-back" >
     <!-- IMU -->
     <xacro:imu_sensor name="${name}_imu" parent="${name}_link" update_rate="100.0">
@@ -61,4 +62,8 @@
       </xacro:sick_tim571_laser>
     </xacro:if>
+    <!-- YDLIDAR TG15 Back -->
+    <xacro:if value="${add_on_module == 'lidar-back'}">
+      <xacro:ydlidar_add_on name="ydlidar" parent="${name}_link"/>
+    </xacro:if>
     <!-- Sonars -->
     <xacro:if value="${has_sonars}">
