Commit message: Fixed wrong inertia calculation in URDF

File: pmb2_description/urdf/sensors/ydlidar_tg15_laser.urdf.xacro (robot description, xacro)
@@ -17,5 +17,5 @@
     <link name="${name}_link" type="laser">
       <inertial>
-        <origin xyz="0.0 0.0 0.0" rpy="0 0 0"/>
+        <origin xyz="-0.000027 0 0.016948" rpy="0 0 0"/>
         <mass value="0.175"/>
         <inertia ixx="0.000074433" ixy="-1.585e-14" ixz="-0.000000073" iyy="0.000074641" iyz="1.714e-14" izz="0.000113319"/>

File: pmb2_description/urdf/ydlidar_add_on/ydlidar_add_on.urdf.xacro (robot description, xacro)
@@ -19,10 +19,10 @@
     <link name="${name}_add_on_link">
       <inertial>
-        <origin xyz="0.0 0.0 0.0" rpy="0.0 0.0 0.0"/>
+        <origin xyz="0.057577 0.001831 -0.007628" rpy="0.0 0.0 0.0"/>
         <mass value="0.152"/>
-        <inertia ixx="0.00690488876" ixy="0.000073254" ixz="0.0076684" iyy="0.015874966" iyz="-0.000049362" izz="0.010290654"/>
+        <inertia ixx="0.000669815" ixy="0.000003921" ixz="0.000005377" iyy="0.000221633" iyz="0.000007046" izz="0.000871373"/>
       </inertial>
       <visual>
-        <origin xyz="0.30631686 0.0 -0.210" rpy="0 0 0"/>
+        <origin xyz="0.0 0.0 0.0" rpy="0 0 0"/>
         <geometry>
           <mesh filename="package://pmb2_description/meshes/ydlidar_add_on/ydlidar_add_on.stl" scale="1 1 1"/>
@@ -31,5 +31,5 @@
       </visual>
       <collision>
-        <origin xyz="0.30631686 0.0 -0.210" rpy="0 0 0" />
+        <origin xyz="0.0 0.0 0.0" rpy="0 0 0" />
         <geometry>
           <mesh filename="package://pmb2_description/meshes/ydlidar_add_on/ydlidar_add_on.stl" scale="1 1 1"/>
