Commit message: Realistic ydlidar properties

File: pmb2_description/urdf/base/base_sensors.urdf.xacro (robot description, xacro)
@@ -64,5 +64,5 @@
     <!-- YDLIDAR TG15 Back -->
     <xacro:if value="${add_on_module == 'lidar-back'}">
-      <xacro:ydlidar_add_on name="ydlidar" parent="${name}_link"/>
+      <xacro:ydlidar_add_on name="lidar_back" parent="${name}_link"/>
     </xacro:if>
     <!-- Sonars -->

File: pmb2_description/urdf/sensors/ydlidar_tg15_laser.gazebo.xacro (robot description, xacro)
@@ -23,5 +23,5 @@
             <horizontal>
               <!-- UPDATE FOR ACTUAL YDLIDAR TG15 -->
-              <samples>${818}</samples>
+              <samples>${2000}</samples>              <!-- This should give angular resolution of around 0.18 degrees -->
               <resolution>1</resolution>              <!-- not the sensor resolution; just 1 -->
               <min_angle>${min_angle}</min_angle>
@@ -32,5 +32,5 @@
             <min>0.05</min>
             <max>15.0</max>
-            <resolution>0.001</resolution>
+            <resolution>0.001</resolution>            <!-- rays linear resolution in m -->
           </range>
           <noise>
@@ -45,5 +45,5 @@
           </ros>
           <output_type>sensor_msgs/LaserScan</output_type>
-          <frame_name>${name}_link</frame_name>
+          <frame_name>${name}</frame_name>
         </plugin>
       </sensor>

File: pmb2_description/urdf/sensors/ydlidar_tg15_laser.urdf.xacro (robot description, xacro)
@@ -15,5 +15,5 @@
   <xacro:include filename="$(find pmb2_description)/urdf/sensors/ydlidar_tg15_laser.gazebo.xacro" />
   <xacro:macro name="ydlidar_tg15_laser" params="name parent xyz rpy ros_topic update_rate min_angle max_angle">
-    <link name="${name}_link" type="laser">
+    <link name="${name}" type="laser">
       <inertial>
         <origin xyz="-0.000027 0 0.016948" rpy="0 0 0"/>
@@ -33,5 +33,5 @@
       <origin xyz="${xyz}" rpy="${rpy}"/>
       <parent link="${parent}"/>
-      <child link="${name}_link"/>
+      <child link="${name}"/>
     </joint>
     <!-- gazebo extensions -->

File: pmb2_description/urdf/ydlidar_add_on/ydlidar_add_on.urdf.xacro (robot description, xacro)
@@ -45,5 +45,5 @@
     </joint>
     <!-- Add LIDAR Sensor -->
-    <xacro:ydlidar_tg15_laser name="${name}_link" parent="${name}_add_on_link" xyz="0.0 0.0 0.0" rpy="0.0 0.0 ${180 * deg_to_rad}" ros_topic="scan_raw_back" update_rate="10" min_angle="${-180 * deg_to_rad}" max_angle="${180 * deg_to_rad}">
+    <xacro:ydlidar_tg15_laser name="${name}" parent="${name}_add_on_link" xyz="0.0 0.0 0.0" rpy="0.0 0.0 ${180 * deg_to_rad}" ros_topic="scan_raw_back" update_rate="10" min_angle="${-180 * deg_to_rad}" max_angle="${180 * deg_to_rad}">
     </xacro:ydlidar_tg15_laser>
    </xacro:macro>

Commit message: Uniformed laser frames.

File: pmb2_description/urdf/base/base_sensors.urdf.xacro (robot description, xacro)
@@ -64,5 +64,5 @@
     <!-- YDLIDAR TG15 Back -->
     <xacro:if value="${add_on_module == 'lidar-back'}">
-      <xacro:ydlidar_add_on name="base_laser_back" parent="${name}_link"/>
+      <xacro:ydlidar_add_on name="laser_back" parent="${name}_link"/>
     </xacro:if>
     <!-- Sonars -->

File: pmb2_description/urdf/ydlidar_add_on/ydlidar_add_on.urdf.xacro (robot description, xacro)
@@ -17,5 +17,5 @@
   <!-- MACRO DEFINITION-->
   <xacro:macro name="ydlidar_add_on" params="name parent">
-    <link name="${name}_add_on_link">
+    <link name="${name}_base">
       <inertial>
         <origin xyz="0.057577 0.001831 -0.007628" rpy="0.0 0.0 0.0"/>
@@ -40,10 +40,10 @@
     <joint name="${name}_add_on_joint" type="fixed">
       <parent link="${parent}"/>
-      <child link="${name}_add_on_link"/>
+      <child link="${name}_base"/>
       <origin xyz="-0.30631686 0.0 0.210" rpy="0 0 0" />
       <axis xyz="0 0 1" />
     </joint>
     <!-- Add LIDAR Sensor -->
-    <xacro:ydlidar_tg15_laser name="${name}" parent="${name}_add_on_link" xyz="0.0 0.0 0.0" rpy="0.0 0.0 ${180 * deg_to_rad}" ros_topic="scan_raw_back" update_rate="10" min_angle="${-180 * deg_to_rad}" max_angle="${180 * deg_to_rad}">
+    <xacro:ydlidar_tg15_laser name="${name}_frame" parent="${name}_base" xyz="0.0 0.0 0.0" rpy="0.0 0.0 ${180 * deg_to_rad}" ros_topic="scan_raw_back" update_rate="10" min_angle="${-180 * deg_to_rad}" max_angle="${180 * deg_to_rad}">
     </xacro:ydlidar_tg15_laser>
    </xacro:macro>

Commit message: Fix bug

File: pmb2_description/urdf/base/base_sensors.urdf.xacro (robot description, xacro)
@@ -28,5 +28,5 @@
   <xacro:include filename="$(find pmb2_description)/urdf/ydlidar_add_on/ydlidar_add_on.urdf.xacro" />
   <!-- MACRO DEFINITION -->
-  <xacro:macro name="base_sensors" params="name laser_model:=sick-571 has_sonars:=false has_microphone:=false add_on_module:=lidar-back" >
+  <xacro:macro name="base_sensors" params="name laser_model:=sick-571 has_sonars:=false has_microphone:=false add_on_module:=${add_on_module}" >
     <!-- IMU -->
     <xacro:imu_sensor name="${name}_imu" parent="${name}_link" update_rate="100.0">

Commit message: Fix Bug

File: pmb2_description/urdf/base/base_sensors.urdf.xacro (robot description, xacro)
@@ -28,5 +28,5 @@
   <xacro:include filename="$(find pmb2_description)/urdf/ydlidar_add_on/ydlidar_add_on.urdf.xacro" />
   <!-- MACRO DEFINITION -->
-  <xacro:macro name="base_sensors" params="name laser_model:=sick-571 has_sonars:=false has_microphone:=false add_on_module:=${add_on_module}" >
+  <xacro:macro name="base_sensors" params="name laser_model:=sick-571 has_sonars:=false has_microphone:=false add_on_module:=lidar-back" >
     <!-- IMU -->
     <xacro:imu_sensor name="${name}_imu" parent="${name}_link" update_rate="100.0">

Commit message: Fix laser back frames and sim

File: pmb2_description/urdf/base/base_sensors.urdf.xacro (robot description, xacro)
@@ -64,5 +64,5 @@
     <!-- YDLIDAR TG15 Back -->
     <xacro:if value="${add_on_module == 'lidar-back'}">
-      <xacro:ydlidar_add_on name="laser_back" parent="${name}_link"/>
+      <xacro:ydlidar_add_on name="${name}_laser_back" parent="${name}_link"/>
     </xacro:if>
     <!-- Sonars -->

File: pmb2_description/urdf/sensors/ydlidar_tg15_laser.gazebo.xacro (robot description, xacro)
@@ -45,5 +45,5 @@
           </ros>
           <output_type>sensor_msgs/LaserScan</output_type>
-          <frame_name>${name}</frame_name>
+          <frame_name>${name}_link</frame_name>
         </plugin>
       </sensor>

File: pmb2_description/urdf/sensors/ydlidar_tg15_laser.urdf.xacro (robot description, xacro)
@@ -14,6 +14,6 @@
 <robot xmlns:xacro="http://ros.org/wiki/xacro">
   <xacro:include filename="$(find pmb2_description)/urdf/sensors/ydlidar_tg15_laser.gazebo.xacro" />
-  <xacro:macro name="ydlidar_tg15_laser" params="name parent xyz rpy ros_topic update_rate min_angle max_angle">
-    <link name="${name}" type="laser">
+  <xacro:macro name="ydlidar_tg15_laser" params="name parent *origin ros_topic update_rate min_angle max_angle">
+    <link name="${name}_link" type="laser">
       <inertial>
         <origin xyz="-0.000027 0 0.016948" rpy="0 0 0"/>
@@ -22,5 +22,5 @@
       </inertial>
       <visual>
-        <origin xyz="0.0 0.0 0.0" rpy="0.0 0.0 0.0"/>
+        <origin xyz="0.0 0.0 -0.02" rpy="0.0 0.0 0.0"/>
         <geometry>
           <mesh filename="package://pmb2_description/meshes/sensors/ydlidar_tg15.stl"/>
@@ -31,7 +31,7 @@
     <joint name="${name}_joint" type="fixed">
       <axis xyz="0 1 0"/>
-      <origin xyz="${xyz}" rpy="${rpy}"/>
+      <xacro:insert_block name="origin"/>
       <parent link="${parent}"/>
-      <child link="${name}"/>
+      <child link="${name}_link"/>
     </joint>
     <!-- gazebo extensions -->

File: pmb2_description/urdf/ydlidar_add_on/ydlidar_add_on.urdf.xacro (robot description, xacro)
@@ -17,5 +17,5 @@
   <!-- MACRO DEFINITION-->
   <xacro:macro name="ydlidar_add_on" params="name parent">
-    <link name="${name}_base">
+    <link name="${name}_mount_link">
       <inertial>
         <origin xyz="0.057577 0.001831 -0.007628" rpy="0.0 0.0 0.0"/>
@@ -38,12 +38,13 @@
       </collision>
     </link>
-    <joint name="${name}_add_on_joint" type="fixed">
+    <joint name="${name}_mount_joint" type="fixed">
       <parent link="${parent}"/>
-      <child link="${name}_base"/>
+      <child link="${name}_mount_link"/>
       <origin xyz="-0.30631686 0.0 0.210" rpy="0 0 0" />
       <axis xyz="0 0 1" />
     </joint>
     <!-- Add LIDAR Sensor -->
-    <xacro:ydlidar_tg15_laser name="${name}_frame" parent="${name}_base" xyz="0.0 0.0 0.0" rpy="0.0 0.0 ${180 * deg_to_rad}" ros_topic="scan_raw_back" update_rate="10" min_angle="${-180 * deg_to_rad}" max_angle="${180 * deg_to_rad}">
+    <xacro:ydlidar_tg15_laser name="${name}" parent="${name}_mount_link" ros_topic="scan_raw_back" update_rate="10" min_angle="${-180 * deg_to_rad}" max_angle="${180 * deg_to_rad}">
+      <origin xyz="0.0 0.0 0.02" rpy="0.0 0.0 ${180 * deg_to_rad}" />
     </xacro:ydlidar_tg15_laser>
    </xacro:macro>
