Commit message: Removed collision for yd_lidar_mount

File: pmb2_description/urdf/ydlidar_add_on/ydlidar_add_on.urdf.xacro (robot description, xacro)
@@ -30,11 +30,11 @@
         <material name="Grey" />
       </visual>
-      <collision>
+      <!-- <collision>
         <origin xyz="0.0 0.0 0.0" rpy="0 0 0" />
         <geometry>
-          <mesh filename="package://pmb2_description/meshes/ydlidar_add_on/ydlidar_add_on.stl" scale="1 1 1"/>
+          <mesh filename="package://pmb2_description/meshes/ydlidar_add_on/ydlidar_add_on_collision.dae" scale="1 1 1"/>
         </geometry>
         <material name="Grey" />
-      </collision>
+      </collision> -->
     </link>
     <joint name="${name}_mount_joint" type="fixed">
